Commit message: v1 robotic hand, basically useless...

File: hand.urdf (robot description, URDF)
Before this commit: robot hand, 7 links, 6 joints
Links:
- link Forearm: geometry visual cylinder length=6 radius=2
- link Index: geometry visual cylinder length=4.5 radius=1
- link Middle: geometry visual cylinder length=5 radius=1
- link Palm: geometry visual cylinder length=2 radius=5
- link Pinky: geometry visual cylinder length=3 radius=0.5
- link Ring: geometry visual cylinder length=4 radius=0.7
- link Thumb: geometry visual cylinder length=4 radius=1
Joints:
- joint F1: limit lower=-30 upper=0 effort=1000.0 velocity=0.5 -> lower=-0 upper=1 effort=1000.0 velocity=0.5; origin xyz=0 0 0 rpy=0 0 0 -> xyz=-2 7 0 rpy=1.54 0 0
- joint F2: limit lower=-30 upper=0 effort=1000.0 velocity=0.5 -> lower=-0 upper=1 effort=1000.0 velocity=0.5; origin xyz=0 0 0 rpy=0 0 0 -> xyz=-8.5 3 0 rpy=0.4 1.54 0
- joint F3: limit lower=-30 upper=0 effort=1000.0 velocity=0.5 -> lower=-0 upper=1 effort=1000.0 velocity=0.5; origin xyz=0 0 0 rpy=0 0 0 -> xyz=-9.4 0 0 rpy=0 1.54 0
- joint F4: limit lower=-30 upper=0 effort=1000.0 velocity=0.5 -> lower=-0 upper=1 effort=1000.0 velocity=0.5; origin xyz=0 0 0 rpy=0 0 0 -> xyz=-8 -2.7 0 rpy=-0.4 1.54 0
- joint F5: limit lower=-30 upper=0 effort=1000.0 velocity=0.5 -> lower=-0 upper=1 effort=1000.0 velocity=0.5; origin xyz=0 0 0 rpy=0 0 0 -> xyz=-6.5 -4.5 0 rpy=-0.8 1.54 0
- joint wrist: limit lower=-30 upper=0 effort=1000.0 velocity=0.5 -> lower=-0.26 upper=0.26 effort=1000.0 velocity=0.5; origin xyz=0 0 0 rpy=0 0 0 -> xyz=0 0 0 rpy=0 1.54 0
